File: PBS-HW-LIB/kicad/pbs-scm-bay/pbs-scm-bay.kicad_pcb (KiCad board)
At the start: 2 copper layers, 112 x 32 mm, 10 parts, among them J1 Module receptacle, blind-mate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, J2 Host harness connector, J3 Identity tag pigtail connecto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, J4 Coaxial host antenna port (SC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, SW1 Module-seated switch (signal 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, U1 ESD/TVS protection array (dat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

Commit message: Define the module host connector (PBS-HW-CON-01)
Add PBS-HW-CON-01: a face-to-face blind-mate connector with 17 contacts at
stated positions, flat pads on the module and spring contacts in the bay,
mating order set by four free heights 0.60 mm apart, keyed guide pins
(A 4.00, B 3.00), a bay cover plate and covered module apertures, an SMP
RF contact, forces and electrical ratings. Two dimensioned drawing sheets.

KiCad: both J1 footprints now follow the contact map (module half on the
back of the core board, centred; bay half with spring-contact holes and
guide pins), with 3D models showing contact heights, guide pins and the
cover plate. All geometry comes from tools/connector.py.

PBS-HW-SCM-01 v0.3 references the connector document.
Parts:
- J1: value Module receptacle, blind-mate, shuttered (PBS-HW-SCM-01 Section 5.2) -> Host connector, bay half: spring contacts, cover plate and guide pins (PBS-HW-CON-01); footprint PBS_Generic:J1_Module_receptacle_blind_mate_shuttered_PBS_HW_SCM_01_Section_5_2 -> PBS_Generic:J1_Host_connector_bay_half_spring_contacts_cover_plate_and_guide_pins_PBS_HW_CON
- moved J1 3.50 mm to (106.0, 61.0)
Connections:
- J1 pad 10: RS422_RX_N -> GND
- J1 pad 11: ID_3V3 -> DET_LOOP
- J1 pad 12: GND -> TX+
- J1 pad 13: ID_SCL -> TX-
- J1 pad 14: ID_SDA -> RX+
- J1 pad 15: DET_LOOP -> RX-
- J1 pad 2: CHASSIS -> GND
- J1 pad 4: GND -> CHASSIS
- J1 pad 7: RS422_TX_P -> ID_3V3
- J1 pad 8: RS422_TX_N -> ID_SCL
- J1 pad 9: RS422_RX_P -> ID_SDA
Other:
- board text added: "J1 Host connector, bay half: spring contacts, cover plate and guide pins (PBS-HW-CON-01)"
- board text added: "PBS-HW-SCM-01 BAY INTERFACE rev 0.3"
- board text removed: "J1 Module receptacle, blind-mate, shuttered (PBS-HW-SCM-01 Section 5.2)"
- board text removed: "PBS-HW-SCM-01 BAY INTERFACE rev 0.2"
